Commit message: readyswim for polygon

File: spider_sldasm/urdf/robot.urdf (robot description, URDF)
Before this commit: robot spider_sldasm, 29 links, 28 joints
Links:
- link Link1-1: geometry collision mesh filename=/home/placo_cpg/spider_sldasm/meshes/Link1-1.STL; visual mesh filename=/home/placo_cpg/spider_sldasm/meshes/Link1-1.STL
- link Link1-2: geometry collision mesh filename=/home/placo_cpg/spider_sldasm/meshes/Link1-2.STL; visual mesh filename=/home/placo_cpg/spider_sldasm/meshes/Link1-2.STL
- link Link1-3: geometry collision mesh filename=/home/placo_cpg/spider_sldasm/meshes/Link1-3.STL; visual mesh filename=/home/placo_cpg/spider_sldasm/meshes/Link1-3.STL
- link Link1-4: geometry collision mesh filename=/home/placo_cpg/spider_sldasm/meshes/Link1-4.STL; visual mesh filename=/home/placo_cpg/spider_sldasm/meshes/Link1-4.STL
- link Link1-5: geometry collision mesh filename=/home/placo_cpg/spider_sldasm/meshes/Link1-5.STL; visual mesh filename=/home/placo_cpg/spider_sldasm/meshes/Link1-5.STL
- link Link1-6: geometry collision mesh filename=/home/placo_cpg/spider_sldasm/meshes/Link1-6.STL; visual mesh filename=/home/placo_cpg/spider_sldasm/meshes/Link1-6.STL
- link Link2-1: geometry collision mesh filename=/home/placo_cpg/spider_sldasm/meshes/Link2-1.STL; visual mesh filename=/home/placo_cpg/spider_sldasm/meshes/Link2-1.STL
- link Link2-2: geometry collision mesh filename=/home/placo_cpg/spider_sldasm/meshes/Link2-2.STL; visual mesh filename=/home/placo_cpg/spider_sldasm/meshes/Link2-2.STL
- link Link2-3: geometry collision mesh filename=/home/placo_cpg/spider_sldasm/meshes/Link2-3.STL; visual mesh filename=/home/placo_cpg/spider_sldasm/meshes/Link2-3.STL
- link Link2-4: geometry collision mesh filename=/home/placo_cpg/spider_sldasm/meshes/Link2-4.STL; visual mesh filename=/home/placo_cpg/spider_sldasm/meshes/Link2-4.STL
- link Link2-5: geometry collision mesh filename=/home/placo_cpg/spider_sldasm/meshes/Link2-5.STL; visual mesh filename=/home/placo_cpg/spider_sldasm/meshes/Link2-5.STL
- link Link2-6: geometry collision mesh filename=/home/placo_cpg/spider_sldasm/meshes/Link2-6.STL; visual mesh filename=/home/placo_cpg/spider_sldasm/meshes/Link2-6.STL
- link Link3-1: geometry collision mesh filename=/home/placo_cpg/spider_sldasm/meshes/Link3-1.STL; visual mesh filename=/home/placo_cpg/spider_sldasm/meshes/Link3-1.STL
- link Link3-2: geometry collision mesh filename=/home/placo_cpg/spider_sldasm/meshes/Link3-2.STL; visual mesh filename=/home/placo_cpg/spider_sldasm/meshes/Link3-2.STL
- link Link3-3: geometry collision mesh filename=/home/placo_cpg/spider_sldasm/meshes/Link3-3.STL; visual mesh filename=/home/placo_cpg/spider_sldasm/meshes/Link3-3.STL
- link Link3-4: geometry collision mesh filename=/home/placo_cpg/spider_sldasm/meshes/Link3-4.STL; visual mesh filename=/home/placo_cpg/spider_sldasm/meshes/Link3-4.STL
- link Link3-5: geometry collision mesh filename=/home/placo_cpg/spider_sldasm/meshes/Link3-5.STL; visual mesh filename=/home/placo_cpg/spider_sldasm/meshes/Link3-5.STL
- link Link3-6: geometry collision mesh filename=/home/placo_cpg/spider_sldasm/meshes/Link3-6.STL; visual mesh filename=/home/placo_cpg/spider_sldasm/meshes/Link3-6.STL
- link Link4-1: geometry collision mesh filename=/home/placo_cpg/spider_sldasm/meshes/Link4-1.STL; visual mesh filename=/home/placo_cpg/spider_sldasm/meshes/Link4-1.STL
- link Link4-2: geometry collision mesh filename=/home/placo_cpg/spider_sldasm/meshes/Link4-2.STL; visual mesh filename=/home/placo_cpg/spider_sldasm/meshes/Link4-2.STL
- link Link4-3: geometry collision mesh filename=/home/placo_cpg/spider_sldasm/meshes/Link4-3.STL; visual mesh filename=/home/placo_cpg/spider_sldasm/meshes/Link4-3.STL
- link Link4-4: geometry collision mesh filename=/home/placo_cpg/spider_sldasm/meshes/Link4-4.STL; visual mesh filename=/home/placo_cpg/spider_sldasm/meshes/Link4-4.STL
- link Link4-5: geometry collision mesh filename=/home/placo_cpg/spider_sldasm/meshes/Link4-5.STL; visual mesh filename=/home/placo_cpg/spider_sldasm/meshes/Link4-5.STL
- link Link4-6: geometry collision mesh filename=/home/placo_cpg/spider_sldasm/meshes/Link4-6.STL; visual mesh filename=/home/placo_cpg/spider_sldasm/meshes/Link4-6.STL
- link base_link: geometry collision mesh filename=/home/placo_cpg/spider_sldasm/meshes/base_link.STL; visual mesh filename=/home/placo_cpg/spider_sldasm/meshes/base_link.STL
