Commit message: foot target bug done!!!!

File: spider_sldasm/urdf/robot copy.urdf (robot description, URDF)
Before this commit: robot spider_sldasm, 25 links, 24 joints
Links:
- link Link1-1: geometry collision mesh filename=/home/zenbot-ljl/placo_spider/spider_sldasm/meshes/Link1-1.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; visual mesh filename=/home/zenbot-ljl/placo_spider/spider_sldasm/meshes/Link1-1.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
- link Link1-2: geometry collision mesh filename=/home/zenbot-ljl/placo_spider/spider_sldasm/meshes/Link1-2.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; visual mesh filename=/home/zenbot-ljl/placo_spider/spider_sldasm/meshes/Link1-2.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
- link Link1-3: geometry collision mesh filename=/home/zenbot-ljl/placo_spider/spider_sldasm/meshes/Link1-3.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; visual mesh filename=/home/zenbot-ljl/placo_spider/spider_sldasm/meshes/Link1-3.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
- link Link1-4: geometry collision mesh filename=/home/zenbot-ljl/placo_spider/spider_sldasm/meshes/Link1-4.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; visual mesh filename=/home/zenbot-ljl/placo_spider/spider_sldasm/meshes/Link1-4.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
- link Link1-5: geometry collision mesh filename=/home/zenbot-ljl/placo_spider/spider_sldasm/meshes/Link1-5.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; visual mesh filename=/home/zenbot-ljl/placo_spider/spider_sldasm/meshes/Link1-5.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
- link Link1-6: geometry collision mesh filename=/home/zenbot-ljl/placo_spider/spider_sldasm/meshes/Link1-6.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; visual mesh filename=/home/zenbot-ljl/placo_spider/spider_sldasm/meshes/Link1-6.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
- link Link2-1: geometry collision mesh filename=/home/zenbot-ljl/placo_spider/spider_sldasm/meshes/Link2-1.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; visual mesh filename=/home/zenbot-ljl/placo_spider/spider_sldasm/meshes/Link2-1.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
- link Link2-2: geometry collision mesh filename=/home/zenbot-ljl/placo_spider/spider_sldasm/meshes/Link2-2.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; visual mesh filename=/home/zenbot-ljl/placo_spider/spider_sldasm/meshes/Link2-2.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
- link Link2-3: geometry collision mesh filename=/home/zenbot-ljl/placo_spider/spider_sldasm/meshes/Link2-3.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; visual mesh filename=/home/zenbot-ljl/placo_spider/spider_sldasm/meshes/Link2-3.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
- link Link2-4: geometry collision mesh filename=/home/zenbot-ljl/placo_spider/spider_sldasm/meshes/Link2-4.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; visual mesh filename=/home/zenbot-ljl/placo_spider/spider_sldasm/meshes/Link2-4.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
- link Link2-5: geometry collision mesh filename=/home/zenbot-ljl/placo_spider/spider_sldasm/meshes/Link2-5.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; visual mesh filename=/home/zenbot-ljl/placo_spider/spider_sldasm/meshes/Link2-5.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
- link Link2-6: geometry collision mesh filename=/home/zenbot-ljl/placo_spider/spider_sldasm/meshes/Link2-6.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; visual mesh filename=/home/zenbot-ljl/placo_spider/spider_sldasm/meshes/Link2-6.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
- link Link3-1: geometry collision mesh filename=/home/zenbot-ljl/placo_spider/spider_sldasm/meshes/Link3-1.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; visual mesh filename=/home/zenbot-ljl/placo_spider/spider_sldasm/meshes/Link3-1.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
- link Link3-2: geometry collision mesh filename=/home/zenbot-ljl/placo_spider/spider_sldasm/meshes/Link3-2.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; visual mesh filename=/home/zenbot-ljl/placo_spider/spider_sldasm/meshes/Link3-2.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
- link Link3-3: geometry collision mesh filename=/home/zenbot-ljl/placo_spider/spider_sldasm/meshes/Link3-3.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; visual mesh filename=/home/zenbot-ljl/placo_spider/spider_sldasm/meshes/Link3-3.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
- link Link3-4: geometry collision mesh filename=/home/zenbot-ljl/placo_spider/spider_sldasm/meshes/Link3-4.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; visual mesh filename=/home/zenbot-ljl/placo_spider/spider_sldasm/meshes/Link3-4.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
- link Link3-5: geometry collision mesh filename=/home/zenbot-ljl/placo_spider/spider_sldasm/meshes/Link3-5.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; visual mesh filename=/home/zenbot-ljl/placo_spider/spider_sldasm/meshes/Link3-5.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
- link Link3-6: geometry collision mesh filename=/home/zenbot-ljl/placo_spider/spider_sldasm/meshes/Link3-6.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; visual mesh filename=/home/zenbot-ljl/placo_spider/spider_sldasm/meshes/Link3-6.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
- link Link4-1: geometry collision mesh filename=/home/zenbot-ljl/placo_spider/spider_sldasm/meshes/Link4-1.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; visual mesh filename=/home/zenbot-ljl/placo_spider/spider_sldasm/meshes/Link4-1.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
- link Link4-2: geometry collision mesh filename=/home/zenbot-ljl/placo_spider/spider_sldasm/meshes/Link4-2.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; visual mesh filename=/home/zenbot-ljl/placo_spider/spider_sldasm/meshes/Link4-2.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
- link Link4-3: geometry collision mesh filename=/home/zenbot-ljl/placo_spider/spider_sldasm/meshes/Link4-3.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; visual mesh filename=/home/zenbot-ljl/placo_spider/spider_sldasm/meshes/Link4-3.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
- link Link4-4: geometry collision mesh filename=/home/zenbot-ljl/placo_spider/spider_sldasm/meshes/Link4-4.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; visual mesh filename=/home/zenbot-ljl/placo_spider/spider_sldasm/meshes/Link4-4.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
- link Link4-5: geometry collision mesh filename=/home/zenbot-ljl/placo_spider/spider_sldasm/meshes/Link4-5.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; visual mesh filename=/home/zenbot-ljl/placo_spider/spider_sldasm/meshes/Link4-5.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
- link Link4-6: geometry collision mesh filename=/home/zenbot-ljl/placo_spider/spider_sldasm/meshes/Link4-6.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; visual mesh filename=/home/zenbot-ljl/placo_spider/spider_sldasm/meshes/Link4-6.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
- link base_link: geometry collision mesh filename=/home/zenbot-ljl/placo_spider/spider_sldasm/meshes/base_lin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; visual mesh filename=/home/zenbot-ljl/placo_spider/spider_sldasm/meshes/base_lin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

File: spider_sldasm/urdf/robot.urdf (robot description, URDF)
Before this commit: robot spider_sldasm, 29 links, 28 joints
Links:
- link Link1-1: geometry collision mesh filename=/home/zenbot-ljl/placo_spider/spider_sldasm/meshes/Link1-1.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; visual mesh filename=/home/zenbot-ljl/placo_spider/spider_sldasm/meshes/Link1-1.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
- link Link1-2: geometry collision mesh filename=/home/zenbot-ljl/placo_spider/spider_sldasm/meshes/Link1-2.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; visual mesh filename=/home/zenbot-ljl/placo_spider/spider_sldasm/meshes/Link1-2.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
- link Link1-3: geometry collision mesh filename=/home/zenbot-ljl/placo_spider/spider_sldasm/meshes/Link1-3.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; visual mesh filename=/home/zenbot-ljl/placo_spider/spider_sldasm/meshes/Link1-3.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
- link Link1-4: geometry collision mesh filename=/home/zenbot-ljl/placo_spider/spider_sldasm/meshes/Link1-4.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; visual mesh filename=/home/zenbot-ljl/placo_spider/spider_sldasm/meshes/Link1-4.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
- link Link1-5: geometry collision mesh filename=/home/zenbot-ljl/placo_spider/spider_sldasm/meshes/Link1-5.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; visual mesh filename=/home/zenbot-ljl/placo_spider/spider_sldasm/meshes/Link1-5.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
- link Link1-6: geometry collision mesh filename=/home/zenbot-ljl/placo_spider/spider_sldasm/meshes/Link1-6.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; visual mesh filename=/home/zenbot-ljl/placo_spider/spider_sldasm/meshes/Link1-6.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
- link Link2-1: geometry collision mesh filename=/home/zenbot-ljl/placo_spider/spider_sldasm/meshes/Link2-1.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; visual mesh filename=/home/zenbot-ljl/placo_spider/spider_sldasm/meshes/Link2-1.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
- link Link2-2: geometry collision mesh filename=/home/zenbot-ljl/placo_spider/spider_sldasm/meshes/Link2-2.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; visual mesh filename=/home/zenbot-ljl/placo_spider/spider_sldasm/meshes/Link2-2.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
- link Link2-3: geometry collision mesh filename=/home/zenbot-ljl/placo_spider/spider_sldasm/meshes/Link2-3.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; visual mesh filename=/home/zenbot-ljl/placo_spider/spider_sldasm/meshes/Link2-3.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
- link Link2-4: geometry collision mesh filename=/home/zenbot-ljl/placo_spider/spider_sldasm/meshes/Link2-4.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; visual mesh filename=/home/zenbot-ljl/placo_spider/spider_sldasm/meshes/Link2-4.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
- link Link2-5: geometry collision mesh filename=/home/zenbot-ljl/placo_spider/spider_sldasm/meshes/Link2-5.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; visual mesh filename=/home/zenbot-ljl/placo_spider/spider_sldasm/meshes/Link2-5.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
- link Link2-6: geometry collision mesh filename=/home/zenbot-ljl/placo_spider/spider_sldasm/meshes/Link2-6.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; visual mesh filename=/home/zenbot-ljl/placo_spider/spider_sldasm/meshes/Link2-6.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
- link Link3-1: geometry collision mesh filename=/home/zenbot-ljl/placo_spider/spider_sldasm/meshes/Link3-1.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; visual mesh filename=/home/zenbot-ljl/placo_spider/spider_sldasm/meshes/Link3-1.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
- link Link3-2: geometry collision mesh filename=/home/zenbot-ljl/placo_spider/spider_sldasm/meshes/Link3-2.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; visual mesh filename=/home/zenbot-ljl/placo_spider/spider_sldasm/meshes/Link3-2.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
- link Link3-3: geometry collision mesh filename=/home/zenbot-ljl/placo_spider/spider_sldasm/meshes/Link3-3.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; visual mesh filename=/home/zenbot-ljl/placo_spider/spider_sldasm/meshes/Link3-3.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
- link Link3-4: geometry collision mesh filename=/home/zenbot-ljl/placo_spider/spider_sldasm/meshes/Link3-4.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; visual mesh filename=/home/zenbot-ljl/placo_spider/spider_sldasm/meshes/Link3-4.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
- link Link3-5: geometry collision mesh filename=/home/zenbot-ljl/placo_spider/spider_sldasm/meshes/Link3-5.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; visual mesh filename=/home/zenbot-ljl/placo_spider/spider_sldasm/meshes/Link3-5.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
- link Link3-6: geometry collision mesh filename=/home/zenbot-ljl/placo_spider/spider_sldasm/meshes/Link3-6.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; visual mesh filename=/home/zenbot-ljl/placo_spider/spider_sldasm/meshes/Link3-6.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
- link Link4-1: geometry collision mesh filename=/home/zenbot-ljl/placo_spider/spider_sldasm/meshes/Link4-1.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; visual mesh filename=/home/zenbot-ljl/placo_spider/spider_sldasm/meshes/Link4-1.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
- link Link4-2: geometry collision mesh filename=/home/zenbot-ljl/placo_spider/spider_sldasm/meshes/Link4-2.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; visual mesh filename=/home/zenbot-ljl/placo_spider/spider_sldasm/meshes/Link4-2.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
- link Link4-3: geometry collision mesh filename=/home/zenbot-ljl/placo_spider/spider_sldasm/meshes/Link4-3.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; visual mesh filename=/home/zenbot-ljl/placo_spider/spider_sldasm/meshes/Link4-3.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
- link Link4-4: geometry collision mesh filename=/home/zenbot-ljl/placo_spider/spider_sldasm/meshes/Link4-4.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; visual mesh filename=/home/zenbot-ljl/placo_spider/spider_sldasm/meshes/Link4-4.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
- link Link4-5: geometry collision mesh filename=/home/zenbot-ljl/placo_spider/spider_sldasm/meshes/Link4-5.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; visual mesh filename=/home/zenbot-ljl/placo_spider/spider_sldasm/meshes/Link4-5.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
- link Link4-6: geometry collision mesh filename=/home/zenbot-ljl/placo_spider/spider_sldasm/meshes/Link4-6.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; visual mesh filename=/home/zenbot-ljl/placo_spider/spider_sldasm/meshes/Link4-6.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
- link base_link: geometry collision mesh filename=/home/zenbot-ljl/placo_spider/spider_sldasm/meshes/base_lin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; visual mesh filename=/home/zenbot-ljl/placo_spider/spider_sldasm/meshes/base_lin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
